File: Main.kicad_pcb (KiCad board)
At the start: 2 copper layers, 110 x 33 mm, 7 parts, among them J1 Conn_01x02_Socket, J2 Conn_01x02_Socket, J3 Conn_01x02_Socket, Q1 AO3400A, U2 ESP32-C3_SUPERMINI_TH

Commit message: route
Parts:
- added J4: Conn_01x06_Socket, Connector_JST:JST_XH_B6B-XH-A_1x06_P2.50mm_Vertical, F.Cu at (151.2, 62.8)
- R1: footprint Resistor_THT:R_Axial_DIN0204_L3.6mm_D1.6mm_P7.62mm_Horizontal -> Resistor_SMD:R_0805_2012Metric_Pad1.20x1.40mm_HandSolder
- moved R1 15.3 mm to (143.0, 91.0)
- moved Q1 12.0 mm to (143.0, 87.8), turned to 180 degrees
- moved J1 11.3 mm to (138.5, 90.3), turned to 180 degrees
- moved U1 8.07 mm to (128.7, 70.0)
- moved J2 2.54 mm to (120.0, 85.5), turned to 0 degrees
- turned U2 to 180 degrees
Connections:
- J1 pad 1: Net-(J1-Pin_1) -> GND
- J1 pad 2: GND -> Net-(J1-Pin_2)
- Q1 pad 3: Net-(J1-Pin_1) -> Net-(J1-Pin_2)
- U2 pad 1: unconnected-(U2-GPIO1-Pad1) -> S0
- U2 pad 10: BIN2 -> unconnected-(U2-GPIO10-Pad10)
- U2 pad 2: unconnected-(U2-GPIO2-Pad2) -> S1
- U2 pad 20: FAN -> unconnected-(U2-GPIO20-Pad20)
- U2 pad 3: unconnected-(U2-GPIO3-Pad3) -> S2
- U2 pad 4: unconnected-(U2-GPIO4-Pad4) -> S3
- U2 pad 5: unconnected-(U2-GPIO5-Pad5) -> FAN
- U2 pad 6: unconnected-(U2-GPIO6-Pad6) -> BIN2
- U2 pad 7: AIN1 -> BIN1
- U2 pad 9: BIN1 -> AIN1
Routing:
- net AIN1: track 33.8 -> 67.7 mm
- net AIN2: track 33.8 -> 66.6 mm
- net BIN1: track 34.8 -> 61.0 mm
- net BIN2: track 34.1 -> 59.9 mm
- net S3: track 0.00 -> 20.8 mm
- net FAN: track 28.4 -> 49.0 mm
- net S2: track 0.00 -> 17.2 mm
- net S1: track 0.00 -> 13.7 mm
- net S0: track 0.00 -> 9.98 mm
- net B01: track 70.7 -> 79.3 mm
- net B02: track 70.7 -> 79.3 mm
- net A02: track 13.4 -> 20.5 mm
- net Net-(J1-Pin_1): track 5.85 -> 0.00 mm
- net Net-(J1-Pin_2): track 0.00 -> 3.66 mm
- net A01: track 13.1 -> 13.9 mm
Other:
- outline, holes or cut-outs redrawn
