File: Main.kicad_sch (KiCad schematic)
At the start: 7 parts

Commit message: layout
Parts:
- removed A?: Arduino_Nano_v3.x, Module:Arduino_Nano, symbol MCU_Module:Arduino_Nano_v3.x
- added U2: ESP32-C3_SUPERMINI_TH, ESP32-C3_SUPERMINI_TH:MODULE_ESP32-C3_SUPERMINI_TH, symbol ESP32-C3_SUPERMINI_TH:ESP32-C3_SUPERMINI_TH
- J1, J2, J3: renamed from M?; value Motor_DC -> Conn_01x02_Socket; footprint (none) -> Connector_PinSocket_2.54mm:PinSocket_1x02_P2.54mm_Vertical; symbol Motor:Motor_DC -> Connector:Conn_01x02_Socket
- R1: renamed from R?; footprint (none) -> Resistor_THT:R_Axial_DIN0204_L3.6mm_D1.6mm_P7.62mm_Horizontal
- gave numbers to parts that had none: 1
Connections:
- net AIN1: now also U2.7 (GPIO7)
- net AIN2: now also U2.8 (GPIO8)
- net BIN1: now also U2.9 (GPIO9)
- net BIN2: now also U2.10 (GPIO10)
- net GND: now also J1.2 (Pin_2)
- net VCC: now also Q1.2 (S), U2.G (GND)
- new net +5V: U2.5V

Commit message: route
Parts:
- added J4: Conn_01x06_Socket, Connector_JST:JST_XH_B6B-XH-A_1x06_P2.50mm_Vertical, symbol Connector:Conn_01x06_Socket
- R1: footprint Resistor_THT:R_Axial_DIN0204_L3.6mm_D1.6mm_P7.62mm_Horizontal -> Resistor_SMD:R_0805_2012Metric_Pad1.20x1.40mm_HandSolder
Connections:
- net AIN1: now also U2.9 (GPIO9); no longer U2.7 (GPIO7)
- net BIN1: now also U2.7 (GPIO7); no longer U2.9 (GPIO9)
- net BIN2: now also U2.6 (GPIO6); no longer U2.10 (GPIO10)
- net GND: now also J1.1 (Pin_1), R1.1, J4.1 (Pin_1); no longer J1.2 (Pin_2)
- net at Q1.3 (D): now also J1.2 (Pin_2); no longer J1.1 (Pin_1)
- net FAN: now reaches Q1.1 (G), R1.2
- net FAN: now also U2.5 (GPIO5)
- net S0: now reaches U2.1 (GPIO1)
- net S0: now also J4.6 (Pin_6)
- net S1: now reaches U2.2 (GPIO2)
- net S1: now also J4.5 (Pin_5)
- net S2: now reaches U2.3 (GPIO3)
- net S2: now also J4.4 (Pin_4)
- net S3: now reaches U2.4 (GPIO4)
- net S3: now also J4.3 (Pin_3)
- new net +3.3V: J4.2 (Pin_2)
- no-connect marks 0 -> 1
Other:
- moved on the sheet: J1, R1
